File: AudioInjector.ABS.v1.balanced.preamplifier.kicad_pcb (KiCad board)
At the start: 4 copper layers, 100 x 70.7 mm, 149 parts, among them J3 NC3MAH, J4 NC3MAH, J5 NC3FAH2, J6 NC3FAH2, Q1 MMBT4401, Q2 MMBT4401, Q3 MMBT4401, Q4 MMBT4403, U1 NJM4580E, U2 NJM4580E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

Commit message: Generated and added the gerber files.
Connections:
- L_G_R_OUT_1 pad 1: (no net) -> /BMUTEC
- L_G_R_OUT_1 pad 6: (no net) -> /AMUTEC
- V12s_1 pad 4: (no net) -> /Vph
Other:
- rule pad_to_mask_clearance: 0.051 -> 0
